Commit message: feat: complete SITL simulation with Gazebo world, URDF, and all nodes

File: src/buggy_description/urdf/buggy.urdf.xacro (robot description, xacro)
@@ -1,113 +1,135 @@
 <?xml version="1.0"?>
-<sdf version="1.6">
-  <world name="srm_campus">
-    <!-- Lighting -->
-    <include><uri>model://sun</uri></include>
-    <include><uri>model://ground_plane</uri></include>
-    <!-- Physics -->
-    <physics type="ode">
-      <real_time_update_rate>1000.0</real_time_update_rate>
-      <max_step_size>0.001</max_step_size>
-      <real_time_factor>1</real_time_factor>
-    </physics>
-    <!-- ── Campus buildings ── -->
-    <!-- Main Gate (node: MAIN_GATE at -40, 0) -->
-    <model name="main_gate">
-      <static>true</static>
-      <pose>-40 0 1 0 0 0</pose>
-      <link name="link">
-        <visual name="visual">
-          <geometry><box><size>4 2 2</size></box></geometry>
-          <material><ambient>0.8 0.6 0.2 1</ambient></material>
-        </visual>
-        <collision name="collision">
-          <geometry><box><size>4 2 2</size></box></geometry>
-        </collision>
-      </link>
-    </model>
-    <!-- Library Block (node: LIBRARY at 40, 0) -->
-    <model name="library">
-      <static>true</static>
-      <pose>40 0 2 0 0 0</pose>
-      <link name="link">
-        <visual name="visual">
-          <geometry><box><size>8 6 4</size></box></geometry>
-          <material><ambient>0.2 0.4 0.8 1</ambient></material>
-        </visual>
-        <collision name="collision">
-          <geometry><box><size>8 6 4</size></box></geometry>
-        </collision>
-      </link>
-    </model>
-    <!-- Admin Block (node: ADMIN_BLOCK at 0, 30) -->
-    <model name="admin_block">
-      <static>true</static>
-      <pose>0 30 2.5 0 0 0</pose>
-      <link name="link">
-        <visual name="visual">
-          <geometry><box><size>10 8 5</size></box></geometry>
-          <material><ambient>0.8 0.2 0.2 1</ambient></material>
-        </visual>
-        <collision name="collision">
-          <geometry><box><size>10 8 5</size></box></geometry>
-        </collision>
-      </link>
-    </model>
-    <!-- Canteen (node: CANTEEN at 0, -30) -->
-    <model name="canteen">
-      <static>true</static>
-      <pose>0 -30 1.5 0 0 0</pose>
-      <link name="link">
-        <visual name="visual">
-          <geometry><box><size>6 6 3</size></box></geometry>
-          <material><ambient>0.2 0.8 0.2 1</ambient></material>
-        </visual>
-        <collision name="collision">
-          <geometry><box><size>6 6 3</size></box></geometry>
-        </collision>
-      </link>
-    </model>
-    <!-- Parking (node: PARKING at -40, 30) -->
-    <model name="parking">
-      <static>true</static>
-      <pose>-40 30 0.1 0 0 0</pose>
-      <link name="link">
-        <visual name="visual">
-          <geometry><box><size>12 10 0.2</size></box></geometry>
-          <material><ambient>0.4 0.4 0.4 1</ambient></material>
-        </visual>
-        <collision name="collision">
-          <geometry><box><size>12 10 0.2</size></box></geometry>
-        </collision>
-      </link>
-    </model>
-    <!-- Hub (node: HUB at 0, 0) — central roundabout -->
-    <model name="hub">
-      <static>true</static>
-      <pose>0 0 0.05 0 0 0</pose>
-      <link name="link">
-        <visual name="visual">
-          <geometry><cylinder><radius>5</radius><length>0.1</length></cylinder></geometry>
-          <material><ambient>0.6 0.6 0.6 1</ambient></material>
-        </visual>
-        <collision name="collision">
-          <geometry><cylinder><radius>5</radius><length>0.1</length></cylinder></geometry>
-        </collision>
-      </link>
-    </model>
-    <!-- ── Obstacle for testing ── -->
-    <model name="test_obstacle">
-      <static>true</static>
-      <pose>20 0 0.5 0 0 0</pose>
-      <link name="link">
-        <visual name="visual">
-          <geometry><box><size>1 1 1</size></box></geometry>
-          <material><ambient>1 0 0 1</ambient></material>
-        </visual>
-        <collision name="collision">
-          <geometry><box><size>1 1 1</size></box></geometry>
-        </collision>
-      </link>
-    </model>
-  </world>
-</sdf>
+<robot name="srm_buggy" xmlns:xacro="http://www.ros.org/wiki/xacro">
+  <material name="white"><color rgba="1 1 1 1"/></material>
+  <material name="black"><color rgba="0 0 0 1"/></material>
+  <material name="blue"><color rgba="0.2 0.4 0.8 1"/></material>
+  <material name="grey"><color rgba="0.5 0.5 0.5 1"/></material>
+  <link name="base_link"/>
+  <joint name="chassis_joint" type="fixed">
+    <parent link="base_link"/>
+    <child  link="chassis"/>
+    <origin xyz="-0.1 0 0.15" rpy="0 0 0"/>
+  </joint>
+  <link name="chassis">
+    <visual>
+      <geometry><box size="1.2 0.6 0.25"/></geometry>
+      <material name="blue"/>
+    </visual>
+    <collision>
+      <geometry><box size="1.2 0.6 0.25"/></geometry>
+    </collision>
+    <inertial>
+      <mass value="80.0"/>
+      <inertia ixx="5.0" ixy="0" ixz="0" iyy="10.0" iyz="0" izz="12.0"/>
+    </inertial>
+  </link>
+  <xacro:macro name="wheel" params="name x y">
+    <joint name="${name}_joint" type="continuous">
+      <parent link="base_link"/>
+      <child  link="${name}"/>
+      <origin xyz="${x} ${y} 0" rpy="0 0 0"/>
+      <axis xyz="0 0 1"/>
+    </joint>
+    <link name="${name}">
+      <visual>
+        <geometry><cylinder radius="0.18" length="0.12"/></geometry>
+        <material name="black"/>
+      </visual>
+      <collision>
+        <geometry><cylinder radius="0.18" length="0.12"/></geometry>
+      </collision>
+      <inertial>
+        <mass value="3.0"/>
+        <inertia ixx="0.05" ixy="0" ixz="0" iyy="0.05" iyz="0" izz="0.08"/>
+      </inertial>
+    </link>
+  </xacro:macro>
+  <xacro:wheel name="front_left_wheel"  x=" 0.4" y=" 0.35"/>
+  <xacro:wheel name="front_right_wheel" x=" 0.4" y="-0.35"/>
+  <xacro:wheel name="rear_left_wheel"   x="-0.4" y=" 0.35"/>
+  <xacro:wheel name="rear_right_wheel"  x="-0.4" y="-0.35"/>
+  <joint name="lidar_joint" type="fixed">
+    <parent link="chassis"/>
+    <child  link="lidar_link"/>
+    <origin xyz="0.5 0 0.2" rpy="0 0 0"/>
+  </joint>
+  <link name="lidar_link">
+    <visual>
+      <geometry><cylinder radius="0.05" length="0.08"/></geometry>
+      <material name="grey"/>
+    </visual>
+    <inertial>
+      <mass value="0.2"/>
+      <inertia ixx="0.001" ixy="0" ixz="0" iyy="0.001" iyz="0" izz="0.001"/>
+    </inertial>
+  </link>
+  <joint name="imu_joint" type="fixed">
+    <parent link="chassis"/>
+    <child  link="imu_link"/>
+    <origin xyz="0 0 0.1" rpy="0 0 0"/>
+  </joint>
+  <link name="imu_link">
+    <visual>
+      <geometry><box size="0.05 0.05 0.02"/></geometry>
+      <material name="grey"/>
+    </visual>
+    <inertial>
+      <mass value="0.05"/>
+      <inertia ixx="0.0001" ixy="0" ixz="0" iyy="0.0001" iyz="0" izz="0.0001"/>
+    </inertial>
+  </link>
+  <gazebo>
+    <plugin name="diff_drive" filename="libgazebo_ros_diff_drive.so">
+      <left_joint>rear_left_wheel_joint</left_joint>
+      <right_joint>rear_right_wheel_joint</right_joint>
+      <wheel_separation>0.7</wheel_separation>
+      <wheel_diameter>0.36</wheel_diameter>
+      <max_wheel_torque>200</max_wheel_torque>
+      <max_wheel_acceleration>1.0</max_wheel_acceleration>
+      <command_topic>cmd_vel</command_topic>
+      <publish_odom>true</publish_odom>
+      <publish_odom_tf>true</publish_odom_tf>
+      <publish_wheel_tf>true</publish_wheel_tf>
+      <odometry_topic>odom</odometry_topic>
+      <odometry_frame>odom</odometry_frame>
+      <robot_base_frame>base_link</robot_base_frame>
+    </plugin>
+  </gazebo>
+  <gazebo reference="lidar_link">
+    <sensor name="lidar" type="ray">
+      <always_on>true</always_on>
+      <visualize>true</visualize>
+      <update_rate>10</update_rate>
+      <ray>
+        <scan>
+          <horizontal>
+            <samples>360</samples>
+            <resolution>1</resolution>
+            <min_angle>-3.14159</min_angle>
+            <max_angle>3.14159</max_angle>
+          </horizontal>
+        </scan>
+        <range>
+          <min>0.3</min>
+          <max>30.0</max>
+          <resolution>0.01</resolution>
+        </range>
+      </ray>
+      <plugin name="lidar_plugin" filename="libgazebo_ros_ray_sensor.so">
+        <ros><remapping>~/out:=scan</remapping></ros>
+        <output_type>sensor_msgs/LaserScan</output_type>
+        <frame_name>lidar_link</frame_name>
+      </plugin>
+    </sensor>
+  </gazebo>
+  <gazebo reference="imu_link">
+    <sensor name="imu_sensor" type="imu">
+      <always_on>true</always_on>
+      <update_rate>50</update_rate>
+      <plugin name="imu_plugin" filename="libgazebo_ros_imu_sensor.so">
+        <ros><remapping>~/out:=imu/data</remapping></ros>
+        <frame_name>imu_link</frame_name>
+      </plugin>
+    </sensor>
+  </gazebo>
+</robot>

Commit message: feat: fix URDF wheel geometry and waypoint follower controller

File: src/buggy_description/urdf/buggy.urdf.xacro (robot description, xacro)
@@ -1,25 +1,24 @@
 <?xml version="1.0"?>
 <robot name="srm_buggy" xmlns:xacro="http://www.ros.org/wiki/xacro">
-  <material name="white"><color rgba="1 1 1 1"/></material>
-  <material name="black"><color rgba="0 0 0 1"/></material>
+  <material name="black"><color rgba="0.1 0.1 0.1 1"/></material>
   <material name="blue"><color rgba="0.2 0.4 0.8 1"/></material>
-  <material name="grey"><color rgba="0.5 0.5 0.5 1"/></material>
+  <material name="grey"><color rgba="0.6 0.6 0.6 1"/></material>
   <link name="base_link"/>
   <joint name="chassis_joint" type="fixed">
     <parent link="base_link"/>
-    <child  link="chassis"/>
-    <origin xyz="-0.1 0 0.15" rpy="0 0 0"/>
+    <child link="chassis"/>
+    <origin xyz="0 0 0.18" rpy="0 0 0"/>
   </joint>
   <link name="chassis">
     <visual>
-      <geometry><box size="1.2 0.6 0.25"/></geometry>
+      <geometry><box size="1.0 0.5 0.2"/></geometry>
       <material name="blue"/>
     </visual>
     <collision>
-      <geometry><box size="1.2 0.6 0.25"/></geometry>
+      <geometry><box size="1.0 0.5 0.2"/></geometry>
     </collision>
     <inertial>
-      <mass value="80.0"/>
-      <inertia ixx="5.0" ixy="0" ixz="0" iyy="10.0" iyz="0" izz="12.0"/>
+      <mass value="50.0"/>
+      <inertia ixx="2.0" ixy="0" ixz="0" iyy="6.0" iyz="0" izz="7.0"/>
     </inertial>
   </link>
@@ -27,49 +26,52 @@
     <joint name="${name}_joint" type="continuous">
       <parent link="base_link"/>
-      <child  link="${name}"/>
+      <child link="${name}"/>
       <origin xyz="${x} ${y} 0" rpy="0 0 0"/>
-      <axis xyz="0 0 1"/>
+      <axis xyz="0 1 0"/>
     </joint>
     <link name="${name}">
       <visual>
-        <geometry><cylinder radius="0.18" length="0.12"/></geometry>
+        <geometry><box size="0.15 0.1 0.15"/></geometry>
         <material name="black"/>
       </visual>
       <collision>
-        <geometry><cylinder radius="0.18" length="0.12"/></geometry>
+        <geometry><box size="0.15 0.1 0.15"/></geometry>
       </collision>
       <inertial>
-        <mass value="3.0"/>
-        <inertia ixx="0.05" ixy="0" ixz="0" iyy="0.05" iyz="0" izz="0.08"/>
+        <mass value="2.0"/>
+        <inertia ixx="0.01" ixy="0" ixz="0" iyy="0.01" iyz="0" izz="0.01"/>
       </inertial>
     </link>
   </xacro:macro>
-  <xacro:wheel name="front_left_wheel"  x=" 0.4" y=" 0.35"/>
-  <xacro:wheel name="front_right_wheel" x=" 0.4" y="-0.35"/>
-  <xacro:wheel name="rear_left_wheel"   x="-0.4" y=" 0.35"/>
-  <xacro:wheel name="rear_right_wheel"  x="-0.4" y="-0.35"/>
+  <xacro:wheel name="front_left_wheel"  x=" 0.35" y=" 0.30"/>
+  <xacro:wheel name="front_right_wheel" x=" 0.35" y="-0.30"/>
+  <xacro:wheel name="rear_left_wheel"   x="-0.35" y=" 0.30"/>
+  <xacro:wheel name="rear_right_wheel"  x="-0.35" y="-0.30"/>
   <joint name="lidar_joint" type="fixed">
     <parent link="chassis"/>
-    <child  link="lidar_link"/>
-    <origin xyz="0.5 0 0.2" rpy="0 0 0"/>
+    <child link="lidar_link"/>
+    <origin xyz="0.4 0 0.12" rpy="0 0 0"/>
   </joint>
   <link name="lidar_link">
     <visual>
-      <geometry><cylinder radius="0.05" length="0.08"/></geometry>
+      <geometry><cylinder radius="0.04" length="0.06"/></geometry>
       <material name="grey"/>
     </visual>
+    <collision>
+      <geometry><cylinder radius="0.04" length="0.06"/></geometry>
+    </collision>
     <inertial>
-      <mass value="0.2"/>
-      <inertia ixx="0.001" ixy="0" ixz="0" iyy="0.001" iyz="0" izz="0.001"/>
+      <mass value="0.1"/>
+      <inertia ixx="0.0001" ixy="0" ixz="0" iyy="0.0001" iyz="0" izz="0.0001"/>
     </inertial>
   </link>
   <joint name="imu_joint" type="fixed">
     <parent link="chassis"/>
-    <child  link="imu_link"/>
-    <origin xyz="0 0 0.1" rpy="0 0 0"/>
+    <child link="imu_link"/>
+    <origin xyz="0 0 0.08" rpy="0 0 0"/>
   </joint>
   <link name="imu_link">
     <visual>
-      <geometry><box size="0.05 0.05 0.02"/></geometry>
+      <geometry><box size="0.04 0.04 0.02"/></geometry>
       <material name="grey"/>
     </visual>
@@ -83,8 +85,8 @@
       <left_joint>rear_left_wheel_joint</left_joint>
       <right_joint>rear_right_wheel_joint</right_joint>
-      <wheel_separation>0.7</wheel_separation>
-      <wheel_diameter>0.36</wheel_diameter>
-      <max_wheel_torque>200</max_wheel_torque>
-      <max_wheel_acceleration>1.0</max_wheel_acceleration>
+      <wheel_separation>0.60</wheel_separation>
+      <wheel_diameter>0.30</wheel_diameter>
+      <max_wheel_torque>500</max_wheel_torque>
+      <max_wheel_acceleration>2.0</max_wheel_acceleration>
       <command_topic>cmd_vel</command_topic>
       <publish_odom>true</publish_odom>
