Commit message: fix(coderabbit): address all review suggestions

File: src/buggy_description/urdf/buggy_urdf.xacro (robot description, xacro)
@@ -15,5 +15,7 @@
   <xacro:property name="chassis_width"   value="1.20"/>
   <xacro:property name="chassis_height"  value="0.25"/>
-  <xacro:property name="chassis_z"       value="0.35"/>   <!-- ride height -->
+  <!-- chassis_z = wheel_radius + (chassis_height/2) + 0.04 = 0.26 + 0.125 + 0.04 = 0.425
+       This places the tire bottoms at z=0 (ground plane) so base_footprint is correct. -->
+  <xacro:property name="chassis_z"       value="0.425"/>   <!-- ride height -->
   <!-- Roof canopy -->
   <xacro:property name="roof_length"     value="3.20"/>
@@ -543,5 +545,5 @@
       <publish_odom>true</publish_odom>
       <publish_odom_tf>true</publish_odom_tf>
-      <publish_wheel_tf>true</publish_wheel_tf>
+      <publish_wheel_tf>false</publish_wheel_tf>
       <odometry_frame>odom</odometry_frame>
       <robot_base_frame>base_footprint</robot_base_frame>

Commit message: feat: complete navigation circuit — buggy reaches all destinations

File: src/buggy_description/urdf/buggy_urdf.xacro (robot description, xacro)
@@ -590,5 +590,5 @@
       </inertial>
     </link>
-    <gazebo reference="${name}"><mu1>1.0</mu1><mu2>1.0</mu2><kp>1e6</kp><kd>100</kd><material>Gazebo/Black</material></gazebo>
+<gazebo reference="${name}"><mu1>5.0</mu1><mu2>5.0</mu2><kp>1e7</kp><kd>1</kd><minDepth>0.001</minDepth><maxVel>0.1</maxVel><material>Gazebo/Black</material></gazebo>
   </xacro:macro>
   <xacro:wheel name="wfl" px=" 1.30" py=" 0.55" side=" 1"/>
